Commit message: training

File: legged_gym/resources/robots/jamal/urdf/jamal_tested.urdf (robot description, URDF)
Before this commit: robot jamal_description, 18 links, 17 joints
Joints:
- joint FL_calf_joint: limit lower=-2.7227 upper=-0.83776 effort=100 velocity=8 -> lower=-2.7227 upper=-0.83776 effort=100 velocity=20.07
- joint FL_hip_joint: limit lower=-0.17 upper=0.17 effort=100 velocity=8 -> lower=-0.53 upper=0.53 effort=100 velocity=8
- joint FL_thigh_joint: limit lower=-0.5236 upper=1.571 effort=100 velocity=8 -> lower=-1.5708 upper=3.4907 effort=100 velocity=8
- joint FR_calf_joint: limit lower=-2.7227 upper=-0.83776 effort=100 velocity=8 -> lower=-2.7227 upper=-0.83776 effort=100 velocity=20.07
- joint FR_hip_joint: limit lower=-0.17 upper=0.17 effort=100 velocity=8 -> lower=-0.53 upper=0.53 effort=100 velocity=8
- joint FR_thigh_joint: limit lower=-0.5236 upper=1.571 effort=100 velocity=8 -> lower=-1.5708 upper=3.4907 effort=100 velocity=8
- joint RL_calf_joint: limit lower=-2.7227 upper=-0.83776 effort=100 velocity=8 -> lower=-2.7227 upper=-0.83776 effort=100 velocity=20.07
- joint RL_hip_joint: limit lower=-0.17 upper=0.17 effort=100 velocity=8 -> lower=-0.53 upper=0.53 effort=100 velocity=8
- joint RL_thigh_joint: limit lower=-0.5236 upper=1.571 effort=100 velocity=8 -> lower=-0.5236 upper=4.5379 effort=100 velocity=8
- joint RR_calf_joint: limit lower=-2.7227 upper=-0.83776 effort=100 velocity=8 -> lower=-2.7227 upper=-0.83776 effort=100 velocity=20.07
- joint RR_hip_joint: limit lower=-0.17 upper=0.17 effort=100 velocity=8 -> lower=-0.53 upper=0.53 effort=100 velocity=8
- joint RR_thigh_joint: limit lower=-0.5236 upper=1.571 effort=100 velocity=8 -> lower=-0.5236 upper=4.5379 effort=100 velocity=8
