Commit message: Finalized codes with best trained policy

File: legged_gym/resources/robots/jamal/urdf/jamal.urdf (robot description, URDF)
Before this commit: robot jamal_description, 18 links, 17 joints
Joints:
- joint FL_hip_joint: limit lower=-0.17 upper=0.17 effort=100 velocity=8 -> lower=-0.43 upper=0.43 effort=100 velocity=8
- joint FR_hip_joint: limit lower=-0.17 upper=0.17 effort=100 velocity=8 -> lower=-0.43 upper=0.43 effort=100 velocity=8
- joint RL_hip_joint: limit lower=-0.17 upper=0.17 effort=100 velocity=8 -> lower=-0.43 upper=0.43 effort=100 velocity=8
- joint RR_hip_joint: limit lower=-0.17 upper=0.17 effort=100 velocity=8 -> lower=-0.43 upper=0.43 effort=100 velocity=8

Commit message: testing 24-11 1

File: legged_gym/resources/robots/jamal/urdf/jamal.urdf (robot description, URDF)
Before this commit: robot jamal_description, 18 links, 17 joints
Links:
- removed link imu
- added link imu_link, mass 0.001
- added link trunk, mass 12.8185384756311; collision box size=0.3762 0.2 0.114; visual mesh filename=../dae/base.dae
- link base: mass 12.8185384756311 -> None; geometry visual box size=0.001 0.001 0.001
Joints:
- added joint floating_base: type fixed, parent base, child trunk, origin xyz=0 0 0 rpy=0 0 0
- joint FL_calf_joint: limit lower=-2.7227 upper=-0.83776 effort=100 velocity=8 -> lower=-2.69653369433 upper=-0.916297857297 effort=100 velocity=8
- joint FL_hip_joint: limit lower=-0.43 upper=0.43 effort=100 velocity=8 -> lower=-0.802851455917 upper=0.802851455917 effort=100 velocity=8; parent base -> trunk
- joint FL_thigh_joint: limit lower=-0.5236 upper=1.571 effort=100 velocity=8 -> lower=-1.0471975512 upper=4.18879020479 effort=100 velocity=8
- joint FR_calf_joint: limit lower=-2.7227 upper=-0.83776 effort=100 velocity=8 -> lower=-2.69653369433 upper=-0.916297857297 effort=100 velocity=8
- joint FR_hip_joint: limit lower=-0.43 upper=0.43 effort=100 velocity=8 -> lower=-0.802851455917 upper=0.802851455917 effort=100 velocity=8; parent base -> trunk
- joint FR_thigh_joint: limit lower=-0.5236 upper=1.571 effort=100 velocity=8 -> lower=-1.0471975512v upper=4.18879020479 effort=100 velocity=8
- joint RL_calf_joint: limit lower=-2.7227 upper=-0.83776 effort=100 velocity=8 -> lower=-2.69653369433 upper=-0.916297857297 effort=100 velocity=8
- joint RL_hip_joint: limit lower=-0.43 upper=0.43 effort=100 velocity=8 -> lower=-0.802851455917 upper=0.802851455917 effort=100 velocity=8; parent base -> trunk
- joint RL_thigh_joint: limit lower=-0.5236 upper=1.571 effort=100 velocity=8 -> lower=-1.0471975512 upper=4.18879020479 effort=100 velocity=8
- joint RR_calf_joint: limit lower=-2.7227 upper=-0.83776 effort=100 velocity=8 -> lower=-2.69653369433 upper=-0.916297857297 effort=100 velocity=8
- joint RR_hip_joint: limit lower=-0.43 upper=0.43 effort=100 velocity=8 -> lower=-0.802851455917 upper=0.802851455917 effort=100 velocity=8; parent base -> trunk
- joint RR_thigh_joint: limit lower=-0.5236 upper=1.571 effort=100 velocity=8 -> lower=-1.0471975512 upper=4.18879020479 effort=100 velocity=8
- joint imu_joint: child imu -> imu_link; parent base -> trunk

File: legged_gym/resources/robots/jamal/urdf/jamal_tested.urdf (robot description, URDF)
Before this commit: robot jamal_description, 18 links, 17 joints
Links:
- removed link imu
- added link imu_link, mass 0.001
Joints:
- joint FL_calf_joint: limit lower=-2.7227 upper=-0.83776 effort=100 velocity=20.07 -> lower=-2.7227 upper=-0.83776 effort=100 velocity=8
- joint FL_hip_joint: limit lower=-0.53 upper=0.53 effort=100 velocity=8 -> lower=-0.43 upper=0.43 effort=100 velocity=8
- joint FL_thigh_joint: limit lower=-1.5708 upper=3.4907 effort=100 velocity=8 -> lower=-0.5236 upper=1.571 effort=100 velocity=8
- joint FR_calf_joint: limit lower=-2.7227 upper=-0.83776 effort=100 velocity=20.07 -> lower=-2.7227 upper=-0.83776 effort=100 velocity=8
- joint FR_hip_joint: limit lower=-0.53 upper=0.53 effort=100 velocity=8 -> lower=-0.43 upper=0.43 effort=100 velocity=8
- joint FR_thigh_joint: limit lower=-1.5708 upper=3.4907 effort=100 velocity=8 -> lower=-0.5236 upper=1.571 effort=100 velocity=8
- joint RL_calf_joint: limit lower=-2.7227 upper=-0.83776 effort=100 velocity=20.07 -> lower=-2.7227 upper=-0.83776 effort=100 velocity=8
- joint RL_hip_joint: limit lower=-0.53 upper=0.53 effort=100 velocity=8 -> lower=-0.43 upper=0.43 effort=100 velocity=8
- joint RL_thigh_joint: limit lower=-0.5236 upper=4.5379 effort=100 velocity=8 -> lower=-0.5236 upper=1.571 effort=100 velocity=8
- joint RR_calf_joint: limit lower=-2.7227 upper=-0.83776 effort=100 velocity=20.07 -> lower=-2.7227 upper=-0.83776 effort=100 velocity=8
- joint RR_hip_joint: limit lower=-0.53 upper=0.53 effort=100 velocity=8 -> lower=-0.43 upper=0.43 effort=100 velocity=8
- joint RR_thigh_joint: limit lower=-0.5236 upper=4.5379 effort=100 velocity=8 -> lower=-0.5236 upper=1.571 effort=100 velocity=8
- joint imu_joint: child imu -> imu_link

Commit message: testing 2-12 1

File: legged_gym/resources/robots/jamal/urdf/jamal.urdf (robot description, URDF)
Before this commit: robot jamal_description, 19 links, 18 joints
Joints:
- joint FL_calf_joint: limit lower=-2.69653369433 upper=-0.916297857297 effort=100 velocity=8 -> lower=-2.69653369433 upper=-0.916297857297 effort=33.5 velocity=28
- joint FL_hip_joint: limit lower=-0.802851455917 upper=0.802851455917 effort=100 velocity=8 -> lower=-0.802851455917 upper=0.802851455917 effort=33.5 velocity=50
- joint FL_thigh_joint: limit lower=-1.0471975512 upper=4.18879020479 effort=100 velocity=8 -> lower=-1.0471975512 upper=4.18879020479 effort=33.5 velocity=28
- joint FR_calf_joint: limit lower=-2.69653369433 upper=-0.916297857297 effort=100 velocity=8 -> lower=-2.69653369433 upper=-0.916297857297 effort=33.5 velocity=28
- joint FR_hip_joint: limit lower=-0.802851455917 upper=0.802851455917 effort=100 velocity=8 -> lower=-0.802851455917 upper=0.802851455917 effort=33.5 velocity=50
- joint FR_thigh_joint: limit lower=-1.0471975512v upper=4.18879020479 effort=100 velocity=8 -> lower=-1.0471975512 upper=4.18879020479 effort=33.5 velocity=28
- joint RL_calf_joint: limit lower=-2.69653369433 upper=-0.916297857297 effort=100 velocity=8 -> lower=-2.69653369433 upper=-0.916297857297 effort=33.5 velocity=28
- joint RL_hip_joint: limit lower=-0.802851455917 upper=0.802851455917 effort=100 velocity=8 -> lower=-0.802851455917 upper=0.802851455917 effort=33.5 velocity=50
- joint RL_thigh_joint: limit lower=-1.0471975512 upper=4.18879020479 effort=100 velocity=8 -> lower=-1.0471975512 upper=4.18879020479 effort=33.5 velocity=28
- joint RR_calf_joint: limit lower=-2.69653369433 upper=-0.916297857297 effort=100 velocity=8 -> lower=-2.69653369433 upper=-0.916297857297 effort=33.5 velocity=28
- joint RR_hip_joint: limit lower=-0.802851455917 upper=0.802851455917 effort=100 velocity=8 -> lower=-0.802851455917 upper=0.802851455917 effort=33.5 velocity=50
- joint RR_thigh_joint: limit lower=-1.0471975512 upper=4.18879020479 effort=100 velocity=8 -> lower=-1.0471975512 upper=4.18879020479 effort=33.5 velocity=28
- joint imu_joint: origin xyz=-0.02557 0 0.04232 rpy=0 0 0 -> xyz=0 0 0 rpy=0 0 0
